Commit message: update push

File: assets/table/table.urdf (robot description, URDF)
Before this commit: robot table, 16 links, 15 joints
Links:
- removed link caster_fl_link
- removed link caster_fl_swivel_link
- removed link caster_fr_link
- removed link caster_fr_swivel_link
- removed link caster_rl_link
- removed link caster_rl_swivel_link
- removed link caster_rr_link
- removed link caster_rr_swivel_link
Joints:
- removed joint caster_fl_joint
- removed joint caster_fl_swivel_joint
- removed joint caster_fr_joint
- removed joint caster_fr_swivel_joint
- removed joint caster_rl_joint
- removed joint caster_rl_swivel_joint
- removed joint caster_rr_joint
- removed joint caster_rr_swivel_joint
